Commit message: Fix rotation problems

File: src/quadrotor_description/description/neuroBEM_no_collision.urdf.xacro (robot description, xacro)
@@ -9,9 +9,9 @@
   <xacro:property name="IZZ" value="0.00436"/>
   <link name="base_link">
-    <inertial>
+    <!-- <inertial>
       <origin rpy="0 0 0" xyz="0 0 0"/>
       <mass value="${MASS}"/>
       <inertia ixx="${IXX}" ixy="0.0" ixz="0.0" iyy="${IYY}" iyz="0.0" izz="${IZZ}"/>
-    </inertial>
+    </inertial>  -->
     <visual>
       <origin rpy="0 0 0" xyz="0 0 0"/>
@@ -19,6 +19,6 @@
         <sphere radius="${0.1*sqrt(ARM_X**2+ARM_Y**2)}"/>
       </geometry>
-      <material name="black">
-        <color rgba="0.0 0.0 0.0 1.0"/>
+      <material name="red">
+        <color rgba="1.0 0.0 0.0 1.0"/>
       </material>
     </visual>
@@ -75,10 +75,4 @@
       </geometry>
     </visual>
-    <collision>
-      <origin rpy="0 0 ${ARM_Z/2}" xyz="0 0 0"/>
-      <geometry>
-        <cylinder radius="${sqrt(ARM_X**2+ARM_Y**2)}" length="${ARM_Z}"/>
-      </geometry>
-    </collision>
   </link>
   <link name="prop0_link">
