Commit message: change dataset testing method

File: src/quadrotor_description/description/neuroBEM.urdf.xacro (robot description, xacro)
@@ -19,4 +19,7 @@
         <sphere radius="${0.1*sqrt(ARM_X**2+ARM_Y**2)}"/>
       </geometry>
+      <material name="grey">
+        <color rgba="0.0 0.0 0.0 1.0"/>
+      </material>
     </visual>
     <!-- Rotor 1 -->

Commit message: thicker urdf

File: src/quadrotor_description/description/neuroBEM.urdf.xacro (robot description, xacro)
@@ -17,8 +17,11 @@
       <origin rpy="0 0 0" xyz="0 0 0"/>
       <geometry>
+        <cylinder radius="${0.2*sqrt(ARM_X**2+ARM_Y**2)}" length="${0.7*ARM_Z}"/>
+      </geometry>
+      <!-- <geometry>
         <sphere radius="${0.1*sqrt(ARM_X**2+ARM_Y**2)}"/>
-      </geometry>
-      <material name="black">
-        <color rgba="0.0 0.0 0.0 1.0"/>
+      </geometry>   -->
+      <material name="gray">
+        <color rgba="0.5 0.5 0.5 0.8"/>
       </material>
     </visual>
@@ -27,5 +30,5 @@
       <origin xyz="${ARM_X/2} ${ARM_Y/2} 0" rpy="0 0 ${-atan(ARM_X/ARM_Y)}"/>
       <geometry>
-        <box size="${0.1* sqrt(ARM_X**2+ARM_Y**2)} ${sqrt(ARM_X**2+ARM_Y**2)} ${0.1*ARM_Z}"/>
+        <box size="${0.15* sqrt(ARM_X**2+ARM_Y**2)} ${sqrt(ARM_X**2+ARM_Y**2)} ${0.5*ARM_Z}"/>
       </geometry>
     </visual>
@@ -33,5 +36,5 @@
       <origin xyz="${ARM_X} ${ARM_Y} ${ARM_Z/2}" rpy="0 0 0"/>
       <geometry>
-        <cylinder radius="${0.1*ARM_Z}" length="${ARM_Z}"/>
+        <cylinder radius="${0.2*ARM_Z}" length="${ARM_Z}"/>
       </geometry>
     </visual>
@@ -40,5 +43,5 @@
       <origin xyz="${-ARM_X/2} ${ARM_Y/2} 0" rpy="0 0 ${-atan(-ARM_X/ARM_Y)}"/>
       <geometry>
-        <box size="${0.1* sqrt(ARM_X**2+ARM_Y**2)} ${sqrt(ARM_X**2+ARM_Y**2)} ${0.1*ARM_Z}"/>
+        <box size="${0.15* sqrt(ARM_X**2+ARM_Y**2)} ${sqrt(ARM_X**2+ARM_Y**2)} ${0.5*ARM_Z}"/>
       </geometry>
     </visual>
@@ -46,5 +49,5 @@
       <origin xyz="${-ARM_X} ${ARM_Y} ${ARM_Z/2}" rpy="0 0 0"/>
       <geometry>
-        <cylinder radius="${0.1*ARM_Z}" length="${ARM_Z}"/>
+        <cylinder radius="${0.2*ARM_Z}" length="${ARM_Z}"/>
       </geometry>
     </visual>
@@ -53,5 +56,5 @@
       <origin xyz="${-ARM_X/2} ${-ARM_Y/2} 0" rpy="0 0 ${-atan(ARM_X/ARM_Y)}"/>
       <geometry>
-        <box size="${0.1* sqrt(ARM_X**2+ARM_Y**2)} ${sqrt(ARM_X**2+ARM_Y**2)} ${0.1*ARM_Z}"/>
+        <box size="${0.15* sqrt(ARM_X**2+ARM_Y**2)} ${sqrt(ARM_X**2+ARM_Y**2)} ${0.5*ARM_Z}"/>
       </geometry>
     </visual>
@@ -59,5 +62,5 @@
       <origin xyz="${-ARM_X} ${-ARM_Y} ${ARM_Z/2}" rpy="0 0 0"/>
       <geometry>
-        <cylinder radius="${0.1*ARM_Z}" length="${ARM_Z}"/>
+        <cylinder radius="${0.2*ARM_Z}" length="${ARM_Z}"/>
       </geometry>
     </visual>
@@ -66,5 +69,5 @@
       <origin xyz="${ARM_X/2} ${-ARM_Y/2} 0" rpy="0 0 ${-atan(-ARM_X/ARM_Y)}"/>
       <geometry>
-        <box size="${0.1* sqrt(ARM_X**2+ARM_Y**2)} ${sqrt(ARM_X**2+ARM_Y**2)} ${0.1*ARM_Z}"/>
+        <box size="${0.15* sqrt(ARM_X**2+ARM_Y**2)} ${sqrt(ARM_X**2+ARM_Y**2)} ${0.5*ARM_Z}"/>
       </geometry>
     </visual>
@@ -72,5 +75,5 @@
       <origin xyz="${ARM_X} ${-ARM_Y} ${ARM_Z/2}" rpy="0 0 0"/>
       <geometry>
-        <cylinder radius="${0.1*ARM_Z}" length="${ARM_Z}"/>
+        <cylinder radius="${0.2*ARM_Z}" length="${ARM_Z}"/>
       </geometry>
     </visual>

Commit message: Add generic quadrotor urdf with xacro macro

File: src/quadrotor_description/description/neuroBEM.urdf.xacro (robot description, xacro)
@@ -1,131 +1,5 @@
 <?xml version="1.0" encoding="utf-8"?>
-<robot xmlns:xacro="http://www.ros.org/wiki/xacro" name="neuroBEM" >
-  <xacro:property name="ARM_X" value="0.078"/>
-  <xacro:property name="ARM_Y" value="0.1"/>
-  <xacro:property name="ARM_Z" value="0.027"/>
-  <xacro:property name="MASS" value="0.772"/>
-  <xacro:property name="IXX" value="0.00254"/>
-  <xacro:property name="IYY" value="0.00214"/>
-  <xacro:property name="IZZ" value="0.00436"/>
-  <link name="base_link">
-    <inertial>
-      <origin rpy="0 0 0" xyz="0 0 0"/>
-      <mass value="${MASS}"/>
-      <inertia ixx="${IXX}" ixy="0.0" ixz="0.0" iyy="${IYY}" iyz="0.0" izz="${IZZ}"/>
-    </inertial>
-    <visual>
-      <origin rpy="0 0 0" xyz="0 0 0"/>
-      <geometry>
-        <cylinder radius="${0.2*sqrt(ARM_X**2+ARM_Y**2)}" length="${0.7*ARM_Z}"/>
-      </geometry>
-      <!-- <geometry>
-        <sphere radius="${0.1*sqrt(ARM_X**2+ARM_Y**2)}"/>
-      </geometry>   -->
-      <material name="gray">
-        <color rgba="0.5 0.5 0.5 0.8"/>
-      </material>
-    </visual>
-    <!-- Rotor 1 -->
-    <visual>
-      <origin xyz="${ARM_X/2} ${ARM_Y/2} 0" rpy="0 0 ${-atan(ARM_X/ARM_Y)}"/>
-      <geometry>
-        <box size="${0.15* sqrt(ARM_X**2+ARM_Y**2)} ${sqrt(ARM_X**2+ARM_Y**2)} ${0.5*ARM_Z}"/>
-      </geometry>
-    </visual>
-    <visual>
-      <origin xyz="${ARM_X} ${ARM_Y} ${ARM_Z/2}" rpy="0 0 0"/>
-      <geometry>
-        <cylinder radius="${0.2*ARM_Z}" length="${ARM_Z}"/>
-      </geometry>
-    </visual>
-    <!-- Rotor 2 -->
-    <visual>
-      <origin xyz="${-ARM_X/2} ${ARM_Y/2} 0" rpy="0 0 ${-atan(-ARM_X/ARM_Y)}"/>
-      <geometry>
-        <box size="${0.15* sqrt(ARM_X**2+ARM_Y**2)} ${sqrt(ARM_X**2+ARM_Y**2)} ${0.5*ARM_Z}"/>
-      </geometry>
-    </visual>
-    <visual>
-      <origin xyz="${-ARM_X} ${ARM_Y} ${ARM_Z/2}" rpy="0 0 0"/>
-      <geometry>
-        <cylinder radius="${0.2*ARM_Z}" length="${ARM_Z}"/>
-      </geometry>
-    </visual>
-    <!-- Rotor 3 -->
-    <visual>
-      <origin xyz="${-ARM_X/2} ${-ARM_Y/2} 0" rpy="0 0 ${-atan(ARM_X/ARM_Y)}"/>
-      <geometry>
-        <box size="${0.15* sqrt(ARM_X**2+ARM_Y**2)} ${sqrt(ARM_X**2+ARM_Y**2)} ${0.5*ARM_Z}"/>
-      </geometry>
-    </visual>
-    <visual>
-      <origin xyz="${-ARM_X} ${-ARM_Y} ${ARM_Z/2}" rpy="0 0 0"/>
-      <geometry>
-        <cylinder radius="${0.2*ARM_Z}" length="${ARM_Z}"/>
-      </geometry>
-    </visual>
-    <!-- Rotor 4 -->
-    <visual>
-      <origin xyz="${ARM_X/2} ${-ARM_Y/2} 0" rpy="0 0 ${-atan(-ARM_X/ARM_Y)}"/>
-      <geometry>
-        <box size="${0.15* sqrt(ARM_X**2+ARM_Y**2)} ${sqrt(ARM_X**2+ARM_Y**2)} ${0.5*ARM_Z}"/>
-      </geometry>
-    </visual>
-    <visual>
-      <origin xyz="${ARM_X} ${-ARM_Y} ${ARM_Z/2}" rpy="0 0 0"/>
-      <geometry>
-        <cylinder radius="${0.2*ARM_Z}" length="${ARM_Z}"/>
-      </geometry>
-    </visual>
-    <collision>
-      <origin rpy="0 0 ${ARM_Z/2}" xyz="0 0 0"/>
-      <geometry>
-        <cylinder radius="${sqrt(ARM_X**2+ARM_Y**2)}" length="${ARM_Z}"/>
-      </geometry>
-    </collision>
-  </link>
-  <link name="prop0_link">
-    <inertial>
-      <origin rpy="0 0 0" xyz="${ARM_X} -${ARM_Y} ${ARM_Z}" />
-      <mass value="0" />
-      <inertia ixx="0" ixy="0" ixz="0" iyy="0" iyz="0" izz="0" />
-    </inertial>
-  </link>
-  <joint name="prop0_joint" type="fixed">
-      <parent link="base_link" />
-      <child link="prop0_link" />
-  </joint>
-  <link name="prop1_link">
-    <inertial>
-      <origin rpy="0 0 0" xyz="${ARM_X} ${ARM_Y} ${ARM_Z}"/>
-      <mass value="0"/>
-      <inertia ixx="0" ixy="0" ixz="0" iyy="0" iyz="0" izz="0"/>
-    </inertial>
-  </link>
-  <joint name="prop1_joint" type="fixed">
-    <parent link="base_link"/>
-    <child link="prop1_link"/>
-  </joint>
-  <link name="prop2_link">
-    <inertial>
-      <origin rpy="0 0 0" xyz="-${ARM_X} ${ARM_Y} ${ARM_Z}"/>
-      <mass value="0"/>
-      <inertia ixx="0" ixy="0" ixz="0" iyy="0" iyz="0" izz="0"/>
-    </inertial>
-  </link>
-  <joint name="prop2_joint" type="fixed">
-    <parent link="base_link"/>
-    <child link="prop2_link"/>
-  </joint>
-  <link name="prop3_link">
-    <inertial>
-      <origin rpy="0 0 0" xyz="-${ARM_X} -${ARM_Y} ${ARM_Z}"/>
-      <mass value="0"/>
-      <inertia ixx="0" ixy="0" ixz="0" iyy="0" iyz="0" izz="0"/>
-    </inertial>
-  </link>
-  <joint name="prop3_joint" type="fixed">
-    <parent link="base_link"/>
-    <child link="prop3_link"/>
-  </joint>
+<robot xmlns:xacro="http://www.ros.org/wiki/xacro" name="neuroBEM">
+    <xacro:include filename="$(find quadrotor_description)/description/generic.xacro" />
+    <xacro:quadrotor_generic ARM_X='0.078' ARM_Y='0.1' ARM_Z='0.027' MASS='0.772' IXX='0.00254' IYY='0.00214' IZZ='0.00436'/>
 </robot>
