Commit message: Improve the scene

File: src/quadrotor_description/description/generic.xacro (robot description, xacro)
@@ -2,5 +2,5 @@
 <robot xmlns:xacro="http://www.ros.org/wiki/xacro">
     <xacro:macro name="quadrotor_generic"
-        params="ARM_X:=0.1 ARM_Y:=0.1 ARM_Z:=0.03 MASS:=1.0 IXX:=0.0025 IYY:=0.0025 IZZ:=0.005">
+        params="ARM_X:=0.1 ARM_Y:=0.1 ARM_Z:=0.03 MASS:=1.0 IXX:=0.0025 IYY:=0.0025 IZZ:=0.005 base_color:='0.5 0.5 0.5 1.0' prop_color:='0.8 0.0 0.0 0.8'">
         <link name="base_link">
             <inertial>
@@ -14,9 +14,6 @@
                     <cylinder radius="${0.2*sqrt(ARM_X**2+ARM_Y**2)}" length="${0.7*ARM_Z}" />
                 </geometry>
-                <!-- <geometry>
-        <sphere radius="${0.1*sqrt(ARM_X**2+ARM_Y**2)}"/>
-      </geometry>   -->
-                <material name="gray">
-                    <color rgba="0.5 0.5 0.5 0.8" />
+                <material name="base_mat">
+                    <color rgba="${base_color}" />
                 </material>
             </visual>
@@ -90,4 +87,13 @@
                 <inertia ixx="0" ixy="0" ixz="0" iyy="0" iyz="0" izz="0" />
             </inertial>
+            <visual>
+                <origin xyz="${ARM_X} -${ARM_Y} ${ARM_Z}" rpy="0.0 0.0 0.0" />
+                <geometry>
+                    <cylinder radius="${0.7*ARM_X}" length="${0.1*ARM_Z}" />
+                </geometry>
+                <material name='prop_mat'>
+                    <color rgba="${prop_color}" />
+                </material>
+            </visual>
         </link>
         <joint name="prop0_joint" type="fixed">
@@ -101,4 +107,13 @@
                 <inertia ixx="0" ixy="0" ixz="0" iyy="0" iyz="0" izz="0" />
             </inertial>
+            <visual>
+                <origin xyz="${ARM_X} ${ARM_Y} ${ARM_Z}" rpy="0.0 0.0 0.0" />
+                <geometry>
+                    <cylinder radius="${0.7*ARM_X}" length="${0.1*ARM_Z}" />
+                </geometry>
+                <material name='prop_mat'>
+                    <color rgba="${prop_color}" />
+                </material>
+            </visual>
         </link>
         <joint name="prop1_joint" type="fixed">
@@ -112,4 +127,13 @@
                 <inertia ixx="0" ixy="0" ixz="0" iyy="0" iyz="0" izz="0" />
             </inertial>
+            <visual>
+                <origin xyz="-${ARM_X} ${ARM_Y} ${ARM_Z}" rpy="0.0 0.0 0.0" />
+                <geometry>
+                    <cylinder radius="${0.7*ARM_X}" length="${0.1*ARM_Z}" />
+                </geometry>
+                <material name='prop_mat'>
+                    <color rgba="${prop_color}" />
+                </material>
+            </visual>
         </link>
         <joint name="prop2_joint" type="fixed">
@@ -123,4 +147,13 @@
                 <inertia ixx="0" ixy="0" ixz="0" iyy="0" iyz="0" izz="0" />
             </inertial>
+            <visual>
+                <origin xyz="-${ARM_X} -${ARM_Y} ${ARM_Z}" rpy="0.0 0.0 0.0" />
+                <geometry>
+                    <cylinder radius="${0.7*ARM_X}" length="${0.1*ARM_Z}" />
+                </geometry>
+                <material name='prop_mat'>
+                    <color rgba="${prop_color}" />
+                </material>
+            </visual>
         </link>
         <joint name="prop3_joint" type="fixed">

File: src/quadrotor_description/description/neuroBEM.urdf.xacro (robot description, xacro)
@@ -2,4 +2,4 @@
 <robot xmlns:xacro="http://www.ros.org/wiki/xacro" name="neuroBEM">
     <xacro:include filename="$(find quadrotor_description)/description/generic.xacro" />
-    <xacro:quadrotor_generic ARM_X='0.078' ARM_Y='0.1' ARM_Z='0.027' MASS='0.772' IXX='0.00254' IYY='0.00214' IZZ='0.00436'/>
+    <xacro:quadrotor_generic ARM_X='0.078' ARM_Y='0.1' ARM_Z='0.027' MASS='0.772' IXX='0.00254' IYY='0.00214' IZZ='0.00436' base_color='0.5 0.5 0.5 0.9' prop_color= '0.2 0.0 0.6 0.95'/>
 </robot>
