Commit message: Add referece path visualizer

File: src/quadrotor_description/description/cf2x.urdf.xacro (robot description, xacro)
@@ -16,5 +16,5 @@
       <origin rpy="0 0 55" xyz="0 0 0"/>
       <geometry>
-        <mesh filename="$(find quadrotor_description)/meshes/cf2.dae" scale=" 1 1 1"/>
+        <mesh filename="$(find quadrotor_description)/meshes/cf2.dae" scale="1 1 1"/>
       </geometry>
       <material name="grey">

Commit message: Add obstacle to the simulated environment

File: src/quadrotor_description/description/cf2x.urdf.xacro (robot description, xacro)
@@ -16,5 +16,5 @@
       <origin rpy="0 0 55" xyz="0 0 0"/>
       <geometry>
-        <mesh filename="$(find quadrotor_description)/meshes/cf2.dae" scale="1 1 1"/>
+        <mesh filename="$(find quadrotor_description)/meshes/cf2.dae" scale="2"/>
       </geometry>
       <material name="grey">

Commit message: fix camera node

File: src/quadrotor_description/description/cf2x.urdf.xacro (robot description, xacro)
@@ -16,5 +16,5 @@
       <origin rpy="0 0 55" xyz="0 0 0"/>
       <geometry>
-        <mesh filename="$(find quadrotor_description)/meshes/cf2.dae" scale="2"/>
+        <mesh filename="$(find quadrotor_description)/meshes/cf2.dae" scale="2 2 2"/>
       </geometry>
       <material name="grey">

Commit message: Separate image visualizer

File: src/quadrotor_description/description/cf2x.urdf.xacro (robot description, xacro)
@@ -16,5 +16,5 @@
       <origin rpy="0 0 55" xyz="0 0 0"/>
       <geometry>
-        <mesh filename="$(find quadrotor_description)/meshes/cf2.dae" scale="2 2 2"/>
+        <mesh filename="$(find quadrotor_description)/meshes/cf2.dae" scale="1 1 1"/>
       </geometry>
       <material name="grey">

File: src/quadrotor_simulation/world/block.urdf.xacro (robot description, xacro)
@@ -2,4 +2,9 @@
 <robot xmlns:xacro="http://www.ros.org/wiki/xacro" name="block">
     <link name="base_link">
+        <inertial>
+            <origin xyz="0.0 0.0 0.0" rpy="0.0 0.0 0.0"/>
+            <mass value="0.0"/>
+            <inertia ixx="0.0" ixy="0.0" ixz="0.0" iyy="0.0" iyz="0.0" izz="0.0"/>
+        </inertial>
         <visual name='v1'>
             <origin rpy="0 0 0" xyz="0 0 0"/>

File: src/quadrotor_simulation/world/hoop.urdf.xacro (robot description, xacro)
@@ -2,8 +2,13 @@
 <robot xmlns:xacro="http://www.ros.org/wiki/xacro" name="hoop">
     <link name="base_link">
+        <inertial>
+            <origin xyz="0.0 0.0 0.0" rpy="0.0 0.0 0.0"/>
+            <mass value="0.0"/>
+            <inertia ixx="0.0" ixy="0.0" ixz="0.0" iyy="0.0" iyz="0.0" izz="0.0"/>
+        </inertial>
         <visual name='v1'>
             <origin rpy="0 0 0" xyz="0 0 0"/>
             <geometry>
-                <mesh filename="$(find quadrotor_simulation)/meshes/hoop.dae" scale="1.0"/>
+                <mesh filename="$(find quadrotor_simulation)/meshes/hoop.dae" scale="1.0 1.0 1.0"/>
             </geometry>
             <material name="blue">

Commit message: High speeeeds

File: src/quadrotor_description/description/cf2x.urdf.xacro (robot description, xacro)
@@ -16,5 +16,5 @@
       <origin rpy="0 0 55" xyz="0 0 0"/>
       <geometry>
-        <mesh filename="$(find quadrotor_description)/meshes/cf2.dae" scale="1 1 1"/>
+        <mesh filename="$(find quadrotor_description)/meshes/cf2.dae" scale="2 2 2"/>
       </geometry>
       <material name="grey">

File: src/quadrotor_simulation/world/hoop.urdf.xacro (robot description, xacro)
@@ -10,5 +10,5 @@
             <origin rpy="0 0 0" xyz="0 0 0"/>
             <geometry>
-                <mesh filename="$(find quadrotor_simulation)/meshes/hoop.dae" scale="1.0 1.0 1.0"/>
+                <mesh filename="$(find quadrotor_simulation)/meshes/hoop.dae" scale="1.5 1.5 1.5"/>
             </geometry>
             <material name="blue">

Commit message: Add ff_state to the physics node

File: src/quadrotor_description/description/cf2x.urdf.xacro (robot description, xacro)
@@ -1,29 +1,97 @@
 <?xml version="1.0" encoding="utf-8"?>
-<robot xmlns:xacro="http://www.ros.org/wiki/xacro" name="cf2">
-  <properties arm="0.0397" kf="3.16e-10" km="7.94e-12" thrust2weight="2.25" max_speed_kmh="30" gnd_eff_coeff="11.36859" prop_radius="2.31348e-2" drag_coeff_xy="9.1785e-7" drag_coeff_z="10.311e-7" dw_coeff_1="2267.18" dw_coeff_2=".16" dw_coeff_3="-.11" />
+<robot xmlns:xacro="http://www.ros.org/wiki/xacro" name="cf2x" >
+  <xacro:property name="ARM_X" value="0.028"/>
+  <xacro:property name="ARM_Y" value="0.028"/>
+  <xacro:property name="ARM_Z" value="0.0"/>
+  <xacro:property name="MASS" value="0.027"/>
+  <xacro:property name="IXX" value="1.4e-5"/>
+  <xacro:property name="IYY" value="1.4e-5"/>
+  <xacro:property name="IZZ" value="2.17e-5"/>
   <link name="base_link">
     <inertial>
       <origin rpy="0 0 0" xyz="0 0 0"/>
-      <mass value="0.027"/>
-      <inertia ixx="1.4e-5" ixy="0.0" ixz="0.0" iyy="1.4e-5" iyz="0.0" izz="2.17e-5"/>
+      <mass value="${MASS}"/>
+      <inertia ixx="${IXX}" ixy="0.0" ixz="0.0" iyy="${IYY}" iyz="0.0" izz="${IZZ}"/>
     </inertial>
-    <!-- links>
-      <carlos url="https://arxiv.org/pdf/1608.05786.pdf" />
-      <julian url="http://mikehamer.info/assets/papers/Crazyflie%20Modelling.pdf" />
-      <mit url="http://groups.csail.mit.edu/robotics-center/public_papers/Landry15.pdf" />
-    </links -->
-    <visual>
-      <origin rpy="0 0 55" xyz="0 0 0"/>
+    <!-- <visual>
+      <origin rpy="0 0 55" xyz="0 0 0.0"/>
       <geometry>
-        <mesh filename="$(find quadrotor_description)/meshes/cf2.dae" scale="2 2 2"/>
+        <mesh filename="$(find quadrotor_description)/meshes/cf2.dae" scale="1.0 1.0 1.0"/>
       </geometry>
       <material name="grey">
         <color rgba=".5 .5 .5 1"/>
       </material>
+    </visual> -->
+    <visual>
+      <origin rpy="0 0 0" xyz="0 0 0"/>
+      <geometry>
+        <sphere radius="${0.1*sqrt(ARM_X**2+ARM_Y**2)}"/>
+      </geometry>
+      <material name="black">
+        <color rgba="0.0 0.0 0.0 1.0"/>
+      </material>
+    </visual>
+    <!-- Rotor 1 -->
+    <visual>
+      <origin xyz="${ARM_X/2} ${ARM_Y/2} 0" rpy="0 0 ${-atan(ARM_X/ARM_Y)}"/>
+      <geometry>
+        <box size="${0.1* sqrt(ARM_X**2+ARM_Y**2)} ${sqrt(ARM_X**2+ARM_Y**2)} ${0.1*ARM_Z}"/>
+      </geometry>
+    </visual>
+    <visual>
+      <origin xyz="${ARM_X} ${ARM_Y} ${ARM_Z/2}" rpy="0 0 0"/>
+      <geometry>
+        <cylinder radius="${0.1*ARM_Z}" length="${ARM_Z}"/>
+      </geometry>
+    </visual>
+    <!-- Rotor 2 -->
+    <visual>
+      <origin xyz="${-ARM_X/2} ${ARM_Y/2} 0" rpy="0 0 ${-atan(-ARM_X/ARM_Y)}"/>
+      <geometry>
+        <box size="${0.1* sqrt(ARM_X**2+ARM_Y**2)} ${sqrt(ARM_X**2+ARM_Y**2)} ${0.1*ARM_Z}"/>
+      </geometry>
+    </visual>
+    <visual>
+      <origin xyz="${-ARM_X} ${ARM_Y} ${ARM_Z/2}" rpy="0 0 0"/>
+      <geometry>
+        <cylinder radius="${0.1*ARM_Z}" length="${ARM_Z}"/>
+      </geometry>
+    </visual>
+    <!-- Rotor 3 -->
+    <visual>
+      <origin xyz="${-ARM_X/2} ${-ARM_Y/2} 0" rpy="0 0 ${-atan(ARM_X/ARM_Y)}"/>
+      <geometry>
+        <box size="${0.1* sqrt(ARM_X**2+ARM_Y**2)} ${sqrt(ARM_X**2+ARM_Y**2)} ${0.1*ARM_Z}"/>
+      </geometry>
+    </visual>
+    <visual>
+      <origin xyz="${-ARM_X} ${-ARM_Y} ${ARM_Z/2}" rpy="0 0 0"/>
+      <geometry>
+        <cylinder radius="${0.1*ARM_Z}" length="${ARM_Z}"/>
+      </geometry>
+    </visual>
+    <!-- Rotor 4 -->
+    <visual>
+      <origin xyz="${ARM_X/2} ${-ARM_Y/2} 0" rpy="0 0 ${-atan(-ARM_X/ARM_Y)}"/>
+      <geometry>
+        <box size="${0.1* sqrt(ARM_X**2+ARM_Y**2)} ${sqrt(ARM_X**2+ARM_Y**2)} ${0.1*ARM_Z}"/>
+      </geometry>
+    </visual>
+    <visual>
+      <origin xyz="${ARM_X} ${-ARM_Y} ${ARM_Z/2}" rpy="0 0 0"/>
+      <geometry>
+        <cylinder radius="${0.1*ARM_Z}" length="${ARM_Z}"/>
+      </geometry>
     </visual>
     <collision>
-      <origin rpy="0 0 0" xyz="0 0 0"/>
+      <origin rpy="0 0 ${ARM_Z/2}" xyz="0 0 0"/>
       <geometry>
-        <cylinder radius=".06" length=".025"/>
+        <cylinder radius="${sqrt(ARM_X**2+ARM_Y**2)}" length="${ARM_Z}"/>
+      </geometry>
+    </collision>
+    <collision>
+      <origin rpy="0 0 ${ARM_Z/2}" xyz="0 0 0"/>
+      <geometry>
+        <cylinder radius="${sqrt(ARM_X**2+ARM_Y**2)}" length="${ARM_Z}"/>
       </geometry>
     </collision>
@@ -31,16 +99,16 @@
   <link name="prop0_link">
     <inertial>
-      <origin rpy="0 0 0" xyz="0.028 0.028 0"/>
-      <mass value="0"/>
-      <inertia ixx="0" ixy="0" ixz="0" iyy="0" iyz="0" izz="0"/>
+      <origin rpy="0 0 0" xyz="${ARM_X} -${ARM_Y} ${ARM_Z}" />
+      <mass value="0" />
+      <inertia ixx="0" ixy="0" ixz="0" iyy="0" iyz="0" izz="0" />
     </inertial>
   </link>
   <joint name="prop0_joint" type="fixed">
-    <parent link="base_link"/>
-    <child link="prop0_link"/>
+      <parent link="base_link" />
+      <child link="prop0_link" />
   </joint>
   <link name="prop1_link">
     <inertial>
-      <origin rpy="0 0 0" xyz="-0.028 0.028 0"/>
+      <origin rpy="0 0 0" xyz="${ARM_X} ${ARM_Y} ${ARM_Z}"/>
       <mass value="0"/>
       <inertia ixx="0" ixy="0" ixz="0" iyy="0" iyz="0" izz="0"/>
@@ -53,5 +121,5 @@
   <link name="prop2_link">
     <inertial>
-      <origin rpy="0 0 0" xyz="-0.028 -0.028 0"/>
+      <origin rpy="0 0 0" xyz="-${ARM_X} ${ARM_Y} ${ARM_Z}"/>
       <mass value="0"/>
       <inertia ixx="0" ixy="0" ixz="0" iyy="0" iyz="0" izz="0"/>
@@ -64,5 +132,5 @@
   <link name="prop3_link">
     <inertial>
-      <origin rpy="0 0 0" xyz="0.028 -0.028 0"/>
+      <origin rpy="0 0 0" xyz="-${ARM_X} -${ARM_Y} ${ARM_Z}"/>
       <mass value="0"/>
       <inertia ixx="0" ixy="0" ixz="0" iyy="0" iyz="0" izz="0"/>
@@ -73,14 +141,3 @@
     <child link="prop3_link"/>
   </joint>
-  <link name="center_of_mass_link">
-    <inertial>
-      <origin rpy="0 0 0" xyz="0 0 0"/>
-      <mass value="0"/>
-      <inertia ixx="0" ixy="0" ixz="0" iyy="0" iyz="0" izz="0"/>
-    </inertial>
-  </link>
-  <joint name="center_of_mass_joint" type="fixed">
-    <parent link="base_link"/>
-    <child link="center_of_mass_link"/>
-  </joint>
 </robot>

Commit message: Change some difault behavior:

File: src/quadrotor_description/description/cf2x.urdf.xacro (robot description, xacro)
@@ -1,143 +1,5 @@
 <?xml version="1.0" encoding="utf-8"?>
-<robot xmlns:xacro="http://www.ros.org/wiki/xacro" name="cf2x" >
-  <xacro:property name="ARM_X" value="0.028"/>
-  <xacro:property name="ARM_Y" value="0.028"/>
-  <xacro:property name="ARM_Z" value="0.0"/>
-  <xacro:property name="MASS" value="0.027"/>
-  <xacro:property name="IXX" value="1.4e-5"/>
-  <xacro:property name="IYY" value="1.4e-5"/>
-  <xacro:property name="IZZ" value="2.17e-5"/>
-  <link name="base_link">
-    <inertial>
-      <origin rpy="0 0 0" xyz="0 0 0"/>
-      <mass value="${MASS}"/>
-      <inertia ixx="${IXX}" ixy="0.0" ixz="0.0" iyy="${IYY}" iyz="0.0" izz="${IZZ}"/>
-    </inertial>
-    <!-- <visual>
-      <origin rpy="0 0 55" xyz="0 0 0.0"/>
-      <geometry>
-        <mesh filename="$(find quadrotor_description)/meshes/cf2.dae" scale="1.0 1.0 1.0"/>
-      </geometry>
-      <material name="grey">
-        <color rgba=".5 .5 .5 1"/>
-      </material>
-    </visual> -->
-    <visual>
-      <origin rpy="0 0 0" xyz="0 0 0"/>
-      <geometry>
-        <sphere radius="${0.1*sqrt(ARM_X**2+ARM_Y**2)}"/>
-      </geometry>
-      <material name="black">
-        <color rgba="0.0 0.0 0.0 1.0"/>
-      </material>
-    </visual>
-    <!-- Rotor 1 -->
-    <visual>
-      <origin xyz="${ARM_X/2} ${ARM_Y/2} 0" rpy="0 0 ${-atan(ARM_X/ARM_Y)}"/>
-      <geometry>
-        <box size="${0.1* sqrt(ARM_X**2+ARM_Y**2)} ${sqrt(ARM_X**2+ARM_Y**2)} ${0.1*ARM_Z}"/>
-      </geometry>
-    </visual>
-    <visual>
-      <origin xyz="${ARM_X} ${ARM_Y} ${ARM_Z/2}" rpy="0 0 0"/>
-      <geometry>
-        <cylinder radius="${0.1*ARM_Z}" length="${ARM_Z}"/>
-      </geometry>
-    </visual>
-    <!-- Rotor 2 -->
-    <visual>
-      <origin xyz="${-ARM_X/2} ${ARM_Y/2} 0" rpy="0 0 ${-atan(-ARM_X/ARM_Y)}"/>
-      <geometry>
-        <box size="${0.1* sqrt(ARM_X**2+ARM_Y**2)} ${sqrt(ARM_X**2+ARM_Y**2)} ${0.1*ARM_Z}"/>
-      </geometry>
-    </visual>
-    <visual>
-      <origin xyz="${-ARM_X} ${ARM_Y} ${ARM_Z/2}" rpy="0 0 0"/>
-      <geometry>
-        <cylinder radius="${0.1*ARM_Z}" length="${ARM_Z}"/>
-      </geometry>
-    </visual>
-    <!-- Rotor 3 -->
-    <visual>
-      <origin xyz="${-ARM_X/2} ${-ARM_Y/2} 0" rpy="0 0 ${-atan(ARM_X/ARM_Y)}"/>
-      <geometry>
-        <box size="${0.1* sqrt(ARM_X**2+ARM_Y**2)} ${sqrt(ARM_X**2+ARM_Y**2)} ${0.1*ARM_Z}"/>
-      </geometry>
-    </visual>
-    <visual>
-      <origin xyz="${-ARM_X} ${-ARM_Y} ${ARM_Z/2}" rpy="0 0 0"/>
-      <geometry>
-        <cylinder radius="${0.1*ARM_Z}" length="${ARM_Z}"/>
-      </geometry>
-    </visual>
-    <!-- Rotor 4 -->
-    <visual>
-      <origin xyz="${ARM_X/2} ${-ARM_Y/2} 0" rpy="0 0 ${-atan(-ARM_X/ARM_Y)}"/>
-      <geometry>
-        <box size="${0.1* sqrt(ARM_X**2+ARM_Y**2)} ${sqrt(ARM_X**2+ARM_Y**2)} ${0.1*ARM_Z}"/>
-      </geometry>
-    </visual>
-    <visual>
-      <origin xyz="${ARM_X} ${-ARM_Y} ${ARM_Z/2}" rpy="0 0 0"/>
-      <geometry>
-        <cylinder radius="${0.1*ARM_Z}" length="${ARM_Z}"/>
-      </geometry>
-    </visual>
-    <collision>
-      <origin rpy="0 0 ${ARM_Z/2}" xyz="0 0 0"/>
-      <geometry>
-        <cylinder radius="${sqrt(ARM_X**2+ARM_Y**2)}" length="${ARM_Z}"/>
-      </geometry>
-    </collision>
-    <collision>
-      <origin rpy="0 0 ${ARM_Z/2}" xyz="0 0 0"/>
-      <geometry>
-        <cylinder radius="${sqrt(ARM_X**2+ARM_Y**2)}" length="${ARM_Z}"/>
-      </geometry>
-    </collision>
-  </link>
-  <link name="prop0_link">
-    <inertial>
-      <origin rpy="0 0 0" xyz="${ARM_X} -${ARM_Y} ${ARM_Z}" />
-      <mass value="0" />
-      <inertia ixx="0" ixy="0" ixz="0" iyy="0" iyz="0" izz="0" />
-    </inertial>
-  </link>
-  <joint name="prop0_joint" type="fixed">
-      <parent link="base_link" />
-      <child link="prop0_link" />
-  </joint>
-  <link name="prop1_link">
-    <inertial>
-      <origin rpy="0 0 0" xyz="${ARM_X} ${ARM_Y} ${ARM_Z}"/>
-      <mass value="0"/>
-      <inertia ixx="0" ixy="0" ixz="0" iyy="0" iyz="0" izz="0"/>
-    </inertial>
-  </link>
-  <joint name="prop1_joint" type="fixed">
-    <parent link="base_link"/>
-    <child link="prop1_link"/>
-  </joint>
-  <link name="prop2_link">
-    <inertial>
-      <origin rpy="0 0 0" xyz="-${ARM_X} ${ARM_Y} ${ARM_Z}"/>
-      <mass value="0"/>
-      <inertia ixx="0" ixy="0" ixz="0" iyy="0" iyz="0" izz="0"/>
-    </inertial>
-  </link>
-  <joint name="prop2_joint" type="fixed">
-    <parent link="base_link"/>
-    <child link="prop2_link"/>
-  </joint>
-  <link name="prop3_link">
-    <inertial>
-      <origin rpy="0 0 0" xyz="-${ARM_X} -${ARM_Y} ${ARM_Z}"/>
-      <mass value="0"/>
-      <inertia ixx="0" ixy="0" ixz="0" iyy="0" iyz="0" izz="0"/>
-    </inertial>
-  </link>
-  <joint name="prop3_joint" type="fixed">
-    <parent link="base_link"/>
-    <child link="prop3_link"/>
-  </joint>
+<robot xmlns:xacro="http://www.ros.org/wiki/xacro" name="neuroBEM">
+    <xacro:include filename="$(find quadrotor_description)/description/generic.xacro" />
+    <xacro:quadrotor_generic ARM_X='0.028' ARM_Y='0.028' ARM_Z='0.002' MASS='0.027' IXX='1.4e-5' IYY='1.4e-5' IZZ='2.17e-5' base_color='0.5 0.5 0.5 0.9' prop_color= '0.2 0.0 0.6 0.95'/>
 </robot>
